File: hardware/1bttn-1poti.sch (EAGLE design)
At the start: 3 parts, among them X2 MC3FAH-0

Commit message: get potis to work...
Parts:
- R1: value PC16-SHM2 -> 10k
Changed lines of the file:
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@@
 <part name="X2" library="con-neutrik_ag" deviceset="MC3?" device="FAH-0"/>
 <part name="S1" library="switch" deviceset="RDT1034" device=""/>
-<part name="R1" library="piher" deviceset="PC16-SHM2" device=""/>
+<part name="R1" library="piher" deviceset="PC16-SHM2" device="" value="10k"/>
 </parts>
 <sheets>
