File: hardware/shield.sch (EAGLE design)
At the start: 38 parts

Commit message: small changes in schematic and layout
Parts:
- PRESET: device pinhead:PINHD-1X4 -> pinhead:PINHD-1X3
- renumbered JP1 to LIGHT
Connections:
- net N.C.: no longer PRESET.4
- net XA0: now also MODULE1.3; no longer MODULE5.3
- net XA1: now also MODULE2.3; no longer MODULE6.3
- net XA2: no longer MODULE1.3
- net XA3: now also MODULE3.3, MODULE4.3; no longer MODULE2.3
- net XA4: now also MODULE5.3; no longer MODULE3.3
- net XA5: now also MODULE6.3; no longer MODULE4.3
- net XD2: now also MODULE6.2; no longer MODULE1.2
- net XD3: now also MODULE5.2; no longer MODULE2.2
- net XD4: now also MODULE4.2; no longer MODULE3.2
- net XD5: now also MODULE3.2; no longer MODULE4.2
- net XD6: now also MODULE2.2; no longer MODULE5.2
- net XD7: now also MODULE1.2; no longer MODULE6.2
Changed lines of the file:
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@@
 <part name="MODULE7" library="pinhead" deviceset="PINHD-1X3" device=""/>
 <part name="MODULE8" library="pinhead" deviceset="PINHD-1X3" device=""/>
-<part name="PRESET" library="pinhead" deviceset="PINHD-1X4" device=""/>
-<part name="JP1" library="pinhead" deviceset="PINHD-1X2" device=""/>
+<part name="LIGHT" library="pinhead" deviceset="PINHD-1X2" device=""/>
 <part name="R24" library="rcl" deviceset="R-EU_" device="0207/7" value="10k"/>
+<part name="PRESET" library="pinhead" deviceset="PINHD-1X3" device=""/>
 </parts>
 <sheets>
@@
 <instance part="MODULE7" gate="A" x="53.34" y="-124.46"/>
 <instance part="MODULE8" gate="A" x="53.34" y="-142.24"/>
-<instance part="PRESET" gate="A" x="5.08" y="-162.56"/>
-<instance part="JP1" gate="G$1" x="53.34" y="-160.02"/>
+<instance part="LIGHT" gate="G$1" x="53.34" y="-160.02"/>
 <instance part="R24" gate="G$1" x="-109.22" y="-185.42"/>
+<instance part="PRESET" gate="A" x="5.08" y="-160.02"/>
 </instances>
 <busses>
@@
 </segment>
 <segment>
-<pinref part="PRESET" gate="A" pin="1"/>
 <wire x1="-17.78" y1="-157.48" x2="2.54" y2="-157.48" width="0.1524" layer="91"/>
 <label x="-17.78" y="-157.48" size="1.778" layer="95"/>
-</segment>
-<segment>
-<pinref part="JP1" gate="G$1" pin="1"/>
+<pinref part="PRESET" gate="A" pin="1"/>
+</segment>
+<segment>
+<pinref part="LIGHT" gate="G$1" pin="1"/>
 <wire x1="30.48" y1="-157.48" x2="50.8" y2="-157.48" width="0.1524" layer="91"/>
 <label x="30.48" y="-157.48" size="1.778" layer="95"/>
@@
 </segment>
 <segment>
-<pinref part="PRESET" gate="A" pin="2"/>
 <wire x1="-17.78" y1="-160.02" x2="2.54" y2="-160.02" width="0.1524" layer="91"/>
 <label x="-17.78" y="-160.02" size="1.778" layer="95"/>
+<pinref part="PRESET" gate="A" pin="2"/>
 </segment>
 </net>
@@
 </segment>
 <segment>
-<pinref part="PRESET" gate="A" pin="3"/>
 <wire x1="-17.78" y1="-162.56" x2="2.54" y2="-162.56" width="0.1524" layer="91"/>
 <label x="-17.78" y="-162.56" size="1.778" layer="95"/>
+<pinref part="PRESET" gate="A" pin="3"/>
 </segment>
 </net>
@@
 </segment>
 <segment>
-<pinref part="MODULE4" gate="A" pin="3"/>
-<wire x1="-17.78" y1="-144.78" x2="2.54" y2="-144.78" width="0.1524" layer="91"/>
-<label x="-17.78" y="-144.78" size="1.778" layer="95"/>
+<pinref part="MODULE6" gate="A" pin="3"/>
+<wire x1="30.48" y1="-109.22" x2="50.8" y2="-109.22" width="0.1524" layer="91"/>
+<label x="30.48" y="-109.22" size="1.778" layer="95"/>
 </segment>
 </net>
@@
 </segment>
 <segment>
-<pinref part="MODULE3" gate="A" pin="3"/>
-<wire x1="-17.78" y1="-127" x2="2.54" y2="-127" width="0.1524" layer="91"/>
-<label x="-17.78" y="-127" size="1.778" layer="95"/>
+<pinref part="MODULE5" gate="A" pin="3"/>
+<wire x1="30.48" y1="-91.44" x2="50.8" y2="-91.44" width="0.1524" layer="91"/>
+<label x="30.48" y="-91.44" size="1.778" layer="95"/>
 </segment>
 </net>
@@
 </segment>
 <segment>
-<pinref part="MODULE2" gate="A" pin="3"/>
-<wire x1="-17.78" y1="-109.22" x2="2.54" y2="-109.22" width="0.1524" layer="91"/>
-<label x="-17.78" y="-109.22" size="1.778" layer="95"/>
+<pinref part="MODULE4" gate="A" pin="3"/>
+<wire x1="-17.78" y1="-144.78" x2="2.54" y2="-144.78" width="0.1524" layer="91"/>
+<label x="-17.78" y="-144.78" size="1.778" layer="95"/>
+</segment>
+<segment>
+<pinref part="MODULE3" gate="A" pin="3"/>
+<wire x1="-17.78" y1="-127" x2="2.54" y2="-127" width="0.1524" layer="91"/>
+<label x="-17.78" y="-127" size="1.778" layer="95"/>
 </segment>
 </net>
@@
 <label x="-50.8" y="-101.6" size="1.778" layer="95"/>
 </segment>
-<segment>
-<pinref part="MODULE1" gate="A" pin="3"/>
-<wire x1="-17.78" y1="-91.44" x2="2.54" y2="-91.44" width="0.1524" layer="91"/>
-<label x="-17.78" y="-91.44" size="1.778" layer="95"/>
-</segment>
 </net>
 <net name="XA1" class="0">
@@
 </segment>
 <segment>
-<pinref part="MODULE6" gate="A" pin="3"/>
-<wire x1="30.48" y1="-109.22" x2="50.8" y2="-109.22" width="0.1524" layer="91"/>
-<label x="30.48" y="-109.22" size="1.778" layer="95"/>
+<pinref part="MODULE2" gate="A" pin="3"/>
+<wire x1="-17.78" y1="-109.22" x2="2.54" y2="-109.22" width="0.1524" layer="91"/>
+<label x="-17.78" y="-109.22" size="1.778" layer="95"/>
 </segment>
 </net>
@@
 </segment>
 <segment>
-<pinref part="MODULE5" gate="A" pin="3"/>
-<wire x1="30.48" y1="-91.44" x2="50.8" y2="-91.44" width="0.1524" layer="91"/>
-<label x="30.48" y="-91.44" size="1.778" layer="95"/>
+<pinref part="MODULE1" gate="A" pin="3"/>
+<wire x1="-17.78" y1="-91.44" x2="2.54" y2="-91.44" width="0.1524" layer="91"/>
+<label x="-17.78" y="-91.44" size="1.778" layer="95"/>
 </segment>
 </net>
@@
 </segment>
 <segment>
+<pinref part="MODULE6" gate="A" pin="2"/>
+<wire x1="30.48" y1="-106.68" x2="50.8" y2="-106.68" width="0.1524" layer="91"/>
+<label x="30.48" y="-106.68" size="1.778" layer="95"/>
+</segment>
+</net>
+<net name="XD3" class="0">
+<segment>
+<pinref part="R11" gate="G$1" pin="2"/>
+<wire x1="-104.14" y1="-170.18" x2="-76.2" y2="-170.18" width="0.1524" layer="91"/>
+<label x="-83.82" y="-170.18" size="1.778" layer="95"/>
+</segment>
+<segment>
+<pinref part="MODULE5" gate="A" pin="2"/>
+<wire x1="30.48" y1="-88.9" x2="50.8" y2="-88.9" width="0.1524" layer="91"/>
+<label x="30.48" y="-88.9" size="1.778" layer="95"/>
+</segment>
+</net>
+<net name="XD4" class="0">
+<segment>
+<wire x1="-114.3" y1="-165.1" x2="-76.2" y2="-165.1" width="0.1524" layer="91"/>
+<pinref part="R10" gate="G$1" pin="2"/>
+<label x="-83.82" y="-165.1" size="1.778" layer="95"/>
+</segment>
+<segment>
+<pinref part="MODULE4" gate="A" pin="2"/>
+<wire x1="-17.78" y1="-142.24" x2="2.54" y2="-142.24" width="0.1524" layer="91"/>
+<label x="-17.78" y="-142.24" size="1.778" layer="95"/>
+</segment>
+</net>
+<net name="XD5" class="0">
+<segment>
+<pinref part="R9" gate="G$1" pin="2"/>
+<wire x1="-104.14" y1="-160.02" x2="-76.2" y2="-160.02" width="0.1524" layer="91"/>
+<label x="-83.82" y="-160.02" size="1.778" layer="95"/>
+</segment>
+<segment>
+<pinref part="MODULE3" gate="A" pin="2"/>
+<wire x1="-17.78" y1="-124.46" x2="2.54" y2="-124.46" width="0.1524" layer="91"/>
+<label x="-17.78" y="-124.46" size="1.778" layer="95"/>
+</segment>
+</net>
+<net name="XD6" class="0">
+<segment>
+<pinref part="R8" gate="G$1" pin="2"/>
+<wire x1="-114.3" y1="-154.94" x2="-76.2" y2="-154.94" width="0.1524" layer="91"/>
+<label x="-83.82" y="-154.94" size="1.778" layer="95"/>
+</segment>
+<segment>
+<pinref part="MODULE2" gate="A" pin="2"/>
+<wire x1="-17.78" y1="-106.68" x2="2.54" y2="-106.68" width="0.1524" layer="91"/>
+<label x="-17.78" y="-106.68" size="1.778" layer="95"/>
+</segment>
+</net>
+<net name="XD7" class="0">
+<segment>
+<pinref part="R7" gate="G$1" pin="2"/>
+<wire x1="-104.14" y1="-149.86" x2="-76.2" y2="-149.86" width="0.1524" layer="91"/>
+<label x="-83.82" y="-149.86" size="1.778" layer="95"/>
+</segment>
+<segment>
 <pinref part="MODULE1" gate="A" pin="2"/>
 <wire x1="-17.78" y1="-88.9" x2="2.54" y2="-88.9" width="0.1524" layer="91"/>
@@
 </segment>
 </net>
-<net name="XD3" class="0">
-<segment>
-<pinref part="R11" gate="G$1" pin="2"/>
-<wire x1="-104.14" y1="-170.18" x2="-76.2" y2="-170.18" width="0.1524" layer="91"/>
-<label x="-83.82" y="-170.18" size="1.778" layer="95"/>
-</segment>
-<segment>
-<pinref part="MODULE2" gate="A" pin="2"/>
-<wire x1="-17.78" y1="-106.68" x2="2.54" y2="-106.68" width="0.1524" layer="91"/>
-<label x="-17.78" y="-106.68" size="1.778" layer="95"/>
-</segment>
-</net>
-<net name="XD4" class="0">
-<segment>
-<wire x1="-114.3" y1="-165.1" x2="-76.2" y2="-165.1" width="0.1524" layer="91"/>
-<pinref part="R10" gate="G$1" pin="2"/>
-<label x="-83.82" y="-165.1" size="1.778" layer="95"/>
-</segment>
-<segment>
-<pinref part="MODULE3" gate="A" pin="2"/>
-<wire x1="-17.78" y1="-124.46" x2="2.54" y2="-124.46" width="0.1524" layer="91"/>
-<label x="-17.78" y="-124.46" size="1.778" layer="95"/>
-</segment>
-</net>
-<net name="XD5" class="0">
-<segment>
-<pinref part="R9" gate="G$1" pin="2"/>
-<wire x1="-104.14" y1="-160.02" x2="-76.2" y2="-160.02" width="0.1524" layer="91"/>
-<label x="-83.82" y="-160.02" size="1.778" layer="95"/>
-</segment>
-<segment>
-<pinref part="MODULE4" gate="A" pin="2"/>
-<wire x1="-17.78" y1="-142.24" x2="2.54" y2="-142.24" width="0.1524" layer="91"/>
-<label x="-17.78" y="-142.24" size="1.778" layer="95"/>
-</segment>
-</net>
-<net name="XD6" class="0">
-<segment>
-<pinref part="R8" gate="G$1" pin="2"/>
-<wire x1="-114.3" y1="-154.94" x2="-76.2" y2="-154.94" width="0.1524" layer="91"/>
-<label x="-83.82" y="-154.94" size="1.778" layer="95"/>
-</segment>
-<segment>
-<pinref part="MODULE5" gate="A" pin="2"/>
-<wire x1="30.48" y1="-88.9" x2="50.8" y2="-88.9" width="0.1524" layer="91"/>
-<label x="30.48" y="-88.9" size="1.778" layer="95"/>
-</segment>
-</net>
-<net name="XD7" class="0">
-<segment>
-<pinref part="R7" gate="G$1" pin="2"/>
-<wire x1="-104.14" y1="-149.86" x2="-76.2" y2="-149.86" width="0.1524" layer="91"/>
-<label x="-83.82" y="-149.86" size="1.778" layer="95"/>
-</segment>
-<segment>
-<pinref part="MODULE6" gate="A" pin="2"/>
-<wire x1="30.48" y1="-106.68" x2="50.8" y2="-106.68" width="0.1524" layer="91"/>
-<label x="30.48" y="-106.68" size="1.778" layer="95"/>
-</segment>
-</net>
 <net name="N.C." class="0">
 <segment>
@@
 <label x="30.48" y="-144.78" size="1.778" layer="95"/>
 </segment>
-<segment>
-<pinref part="PRESET" gate="A" pin="4"/>
-<wire x1="-17.78" y1="-165.1" x2="2.54" y2="-165.1" width="0.1524" layer="91"/>
-<label x="-17.78" y="-165.1" size="1.778" layer="95"/>
-</segment>
 </net>
 <net name="LED" class="0">
 <segment>
-<pinref part="JP1" gate="G$1" pin="2"/>
+<pinref part="LIGHT" gate="G$1" pin="2"/>
 <wire x1="30.48" y1="-160.02" x2="50.8" y2="-160.02" width="0.1524" layer="91"/>
 <label x="30.48" y="-160.02" size="1.778" layer="95"/>

Commit message: get potis to work...
Parts:
- R18, R19, R20, R21, R22, R23: value 100k -> 1k
Changed lines of the file:
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@@
 <part name="ANALOG" library="pinhead" deviceset="PINHD-1X6" device=""/>
 <part name="DIGI2" library="pinhead" deviceset="PINHD-1X10" device=""/>
-<part name="R20" library="rcl" deviceset="R-EU_" device="0207/7" value="100k"/>
-<part name="R21" library="rcl" deviceset="R-EU_" device="0207/7" value="100k"/>
-<part name="R22" library="rcl" deviceset="R-EU_" device="0207/7" value="100k"/>
-<part name="R23" library="rcl" deviceset="R-EU_" device="0207/7" value="100k"/>
-<part name="R19" library="rcl" deviceset="R-EU_" device="0207/7" value="100k"/>
-<part name="R18" library="rcl" deviceset="R-EU_" device="0207/7" value="100k"/>
+<part name="R20" library="rcl" deviceset="R-EU_" device="0207/7" value="1k"/>
+<part name="R21" library="rcl" deviceset="R-EU_" device="0207/7" value="1k"/>
+<part name="R22" library="rcl" deviceset="R-EU_" device="0207/7" value="1k"/>
+<part name="R23" library="rcl" deviceset="R-EU_" device="0207/7" value="1k"/>
+<part name="R19" library="rcl" deviceset="R-EU_" device="0207/7" value="1k"/>
+<part name="R18" library="rcl" deviceset="R-EU_" device="0207/7" value="1k"/>
 <part name="P+1" library="supply1" deviceset="VCC" device=""/>
 <part name="P+2" library="supply1" deviceset="VCC" device=""/>
